File: Chromatic/Chromatic.kicad_pcb (KiCad board)
At the start: 2 copper layers, 199 parts

Commit message: ATA
Parts:
- removed D1, D10, D11, D12, D13, D14, D15, D16, D17, D18, D19, D2, D20, D21, D22, D23, D24, D25, D26, D27, D28, D29, D3, D30, D31, D32, D33, D34, D35, D36, D37, D38, D39, D4, D40, D41, D42, D43, D44, D45, D46, D47, D48, D49, D5, D50, D51, D52, D53, D54, D55, D56, D57, D58, D59, D6, D60, D61, D62, D63, D64, D65, D66, D67, D68, D69, D7, D70, D71, D72, D73, D74, D75, D76, D77, D78, D79, D8, D80, D81, D82, D83, D84, D85, D86, D87, D88, D89, D9, D90, D91, D92, D93, D94, D95, D96, D97, D98, D99: Diode, ScottoKeebs_Components:Diode_DO-35
- removed S1, S10, S11, S12, S13, S14, S15, S16, S17, S18, S19, S2, S20, S21, S22, S23, S24, S25, S26, S27, S28, S29, S3, S30, S31, S32, S33, S34, S35, S36, S37, S38, S39, S4, S40, S41, S42, S43, S44, S45, S46, S47, S48, S49, S5, S50, S51, S52, S53, S54, S55, S56, S57, S58, S59, S6, S60, S61, S62, S63, S64, S65, S66, S67, S68, S69, S7, S70, S71, S72, S73, S74, S75, S76, S77, S78, S79, S8, S80, S81, S82, S83, S84, S85, S86, S87, S88, S89, S9, S90, S91, S92, S93, S94, S95, S96, S97, S98, S99: Keyswitch, ScottoKeebs_MX:MX_PCB_1.00u
- added D_R0C0: ~, ScottoKeebs_Components:Diode_DO-35, F.Cu at (528.7, 42.4)
- added D_R0C1: ~, ScottoKeebs_Components:Diode_DO-35, F.Cu at (528.7, 45.9)
- added D_R0C10: ~, ScottoKeebs_Components:Diode_DO-35, F.Cu at (528.7, 77.9)
- added D_R0C11: ~, ScottoKeebs_Components:Diode_DO-35, F.Cu at (528.7, 81.4)
- added D_R0C12: ~, ScottoKeebs_Components:Diode_DO-35, F.Cu at (528.7, 85.0)
- added D_R0C13: ~, ScottoKeebs_Components:Diode_DO-35, F.Cu at (539.5, 42.4)
- added D_R0C14: ~, ScottoKeebs_Components:Diode_DO-35, F.Cu at (539.5, 45.9)
- added D_R0C15: ~, ScottoKeebs_Components:Diode_DO-35, F.Cu at (539.5, 49.5)
- added D_R0C16: ~, ScottoKeebs_Components:Diode_DO-35, F.Cu at (539.5, 53.0)
- added D_R0C2: ~, ScottoKeebs_Components:Diode_DO-35, F.Cu at (528.7, 49.5)
- added D_R0C3: ~, ScottoKeebs_Components:Diode_DO-35, F.Cu at (528.7, 53.0)
- added D_R0C4: ~, ScottoKeebs_Components:Diode_DO-35, F.Cu at (528.7, 56.6)
- added D_R0C5: ~, ScottoKeebs_Components:Diode_DO-35, F.Cu at (528.7, 60.1)
- added D_R0C6: ~, ScottoKeebs_Components:Diode_DO-35, F.Cu at (528.7, 63.7)
- added D_R0C7: ~, ScottoKeebs_Components:Diode_DO-35, F.Cu at (528.7, 67.2)
- added D_R0C8: ~, ScottoKeebs_Components:Diode_DO-35, F.Cu at (528.7, 70.8)
- added D_R0C9: ~, ScottoKeebs_Components:Diode_DO-35, F.Cu at (528.7, 74.3)
- added D_R1C0: ~, ScottoKeebs_Components:Diode_DO-35, F.Cu at (539.5, 56.6)
- added D_R1C1: ~, ScottoKeebs_Components:Diode_DO-35, F.Cu at (539.5, 60.1)
- added D_R1C10: ~, ScottoKeebs_Components:Diode_DO-35, F.Cu at (550.2, 45.9)
- added D_R1C11: ~, ScottoKeebs_Components:Diode_DO-35, F.Cu at (550.2, 49.5)
- added D_R1C12: ~, ScottoKeebs_Components:Diode_DO-35, F.Cu at (550.2, 53.0)
- added D_R1C13: ~, ScottoKeebs_Components:Diode_DO-35, F.Cu at (550.2, 56.6)
- added D_R1C14: ~, ScottoKeebs_Components:Diode_DO-35, F.Cu at (550.2, 60.1)
- added D_R1C15: ~, ScottoKeebs_Components:Diode_DO-35, F.Cu at (550.2, 63.7)
- added D_R1C16: ~, ScottoKeebs_Components:Diode_DO-35, F.Cu at (550.2, 67.2)
- added D_R1C2: ~, ScottoKeebs_Components:Diode_DO-35, F.Cu at (539.5, 63.7)
- added D_R1C3: ~, ScottoKeebs_Components:Diode_DO-35, F.Cu at (539.5, 67.2)
- added D_R1C4: ~, ScottoKeebs_Components:Diode_DO-35, F.Cu at (539.5, 70.8)
- added D_R1C5: ~, ScottoKeebs_Components:Diode_DO-35, F.Cu at (539.5, 74.3)
- added D_R1C6: ~, ScottoKeebs_Components:Diode_DO-35, F.Cu at (539.5, 77.9)
- added D_R1C7: ~, ScottoKeebs_Components:Diode_DO-35, F.Cu at (539.5, 81.4)
- added D_R1C8: ~, ScottoKeebs_Components:Diode_DO-35, F.Cu at (539.5, 85.0)
- added D_R1C9: ~, ScottoKeebs_Components:Diode_DO-35, F.Cu at (550.2, 42.4)
- added D_R2C0: ~, ScottoKeebs_Components:Diode_DO-35, F.Cu at (550.2, 70.8)
- added D_R2C1: ~, ScottoKeebs_Components:Diode_DO-35, F.Cu at (550.2, 74.3)
- added D_R2C10: ~, ScottoKeebs_Components:Diode_DO-35, F.Cu at (561.0, 60.1)
- added D_R2C11: ~, ScottoKeebs_Components:Diode_DO-35, F.Cu at (561.0, 63.7)
- added D_R2C12: ~, ScottoKeebs_Components:Diode_DO-35, F.Cu at (561.0, 67.2)
- added D_R2C13: ~, ScottoKeebs_Components:Diode_DO-35, F.Cu at (561.0, 70.8)
- added D_R2C14: ~, ScottoKeebs_Components:Diode_DO-35, F.Cu at (561.0, 74.3)
- added D_R2C15: ~, ScottoKeebs_Components:Diode_DO-35, F.Cu at (561.0, 77.9)
- added D_R2C16: ~, ScottoKeebs_Components:Diode_DO-35, F.Cu at (561.0, 81.4)
- added D_R2C2: ~, ScottoKeebs_Components:Diode_DO-35, F.Cu at (550.2, 77.9)
- added D_R2C3: ~, ScottoKeebs_Components:Diode_DO-35, F.Cu at (550.2, 81.4)
- added D_R2C4: ~, ScottoKeebs_Components:Diode_DO-35, F.Cu at (550.2, 85.0)
- added D_R2C5: ~, ScottoKeebs_Components:Diode_DO-35, F.Cu at (561.0, 42.4)
- added D_R2C6: ~, ScottoKeebs_Components:Diode_DO-35, F.Cu at (561.0, 45.9)
- added D_R2C7: ~, ScottoKeebs_Components:Diode_DO-35, F.Cu at (561.0, 49.5)
- added D_R2C8: ~, ScottoKeebs_Components:Diode_DO-35, F.Cu at (561.0, 53.0)
- added D_R2C9: ~, ScottoKeebs_Components:Diode_DO-35, F.Cu at (561.0, 56.6)
- added SW_0_R0C0: Keyswitch, ScottoKeebs_Hotswap:Hotswap_MX_1.00u, F.Cu at (9.50, 9.50)
- added SW_0_R0C1: Keyswitch, ScottoKeebs_Hotswap:Hotswap_MX_1.00u, F.Cu at (9.50, 28.5)
- added SW_0_R0C10: Keyswitch, ScottoKeebs_Hotswap:Hotswap_MX_1.00u, F.Cu at (9.50, 199.5)
- added SW_0_R0C11: Keyswitch, ScottoKeebs_Hotswap:Hotswap_MX_1.00u, F.Cu at (9.50, 218.5)
- added SW_0_R0C12: Keyswitch, ScottoKeebs_Hotswap:Hotswap_MX_1.00u, F.Cu at (9.50, 237.5)
- added SW_0_R0C13: Keyswitch, ScottoKeebs_Hotswap:Hotswap_MX_1.00u, F.Cu at (9.50, 256.5)
- added SW_0_R0C14: Keyswitch, ScottoKeebs_Hotswap:Hotswap_MX_1.00u, F.Cu at (9.50, 275.5)
- added SW_0_R0C15: Keyswitch, ScottoKeebs_Hotswap:Hotswap_MX_1.00u, F.Cu at (9.50, 294.5)
- added SW_0_R0C16: Keyswitch, ScottoKeebs_Hotswap:Hotswap_MX_1.00u, F.Cu at (9.50, 313.5)
- added SW_0_R0C2: Keyswitch, ScottoKeebs_Hotswap:Hotswap_MX_1.00u, F.Cu at (9.50, 47.5)
- added SW_0_R0C3: Keyswitch, ScottoKeebs_Hotswap:Hotswap_MX_1.00u, F.Cu at (9.50, 66.5)
- added SW_0_R0C4: Keyswitch, ScottoKeebs_Hotswap:Hotswap_MX_1.00u, F.Cu at (9.50, 85.5)
- added SW_0_R0C5: Keyswitch, ScottoKeebs_Hotswap:Hotswap_MX_1.00u, F.Cu at (9.50, 104.5)
- added SW_0_R0C6: Keyswitch, ScottoKeebs_Hotswap:Hotswap_MX_1.00u, F.Cu at (9.50, 123.5)
- added SW_0_R0C7: Keyswitch, ScottoKeebs_Hotswap:Hotswap_MX_1.00u, F.Cu at (9.50, 142.5)
- added SW_0_R0C8: Keyswitch, ScottoKeebs_Hotswap:Hotswap_MX_1.00u, F.Cu at (9.50, 161.5)
- added SW_0_R0C9: Keyswitch, ScottoKeebs_Hotswap:Hotswap_MX_1.00u, F.Cu at (9.50, 180.5)
- added SW_1_R1C0: Keyswitch, ScottoKeebs_Hotswap:Hotswap_MX_1.00u, F.Cu at (28.5, 19.0)
- added SW_1_R1C1: Keyswitch, ScottoKeebs_Hotswap:Hotswap_MX_1.00u, F.Cu at (28.5, 38.0)
- added SW_1_R1C10: Keyswitch, ScottoKeebs_Hotswap:Hotswap_MX_1.00u, F.Cu at (28.5, 209.0)
- added SW_1_R1C11: Keyswitch, ScottoKeebs_Hotswap:Hotswap_MX_1.00u, F.Cu at (28.5, 228.0)
- added SW_1_R1C12: Keyswitch, ScottoKeebs_Hotswap:Hotswap_MX_1.00u, F.Cu at (28.5, 247.0)
- added SW_1_R1C13: Keyswitch, ScottoKeebs_Hotswap:Hotswap_MX_1.00u, F.Cu at (28.5, 266.0)
- added SW_1_R1C14: Keyswitch, ScottoKeebs_Hotswap:Hotswap_MX_1.00u, F.Cu at (28.5, 285.0)
- added SW_1_R1C15: Keyswitch, ScottoKeebs_Hotswap:Hotswap_MX_1.00u, F.Cu at (28.5, 304.0)
- added SW_1_R1C2: Keyswitch, ScottoKeebs_Hotswap:Hotswap_MX_1.00u, F.Cu at (28.5, 57.0)
- added SW_1_R1C3: Keyswitch, ScottoKeebs_Hotswap:Hotswap_MX_1.00u, F.Cu at (28.5, 76.0)
- added SW_1_R1C4: Keyswitch, ScottoKeebs_Hotswap:Hotswap_MX_1.00u, F.Cu at (28.5, 95.0)
- added SW_1_R1C5: Keyswitch, ScottoKeebs_Hotswap:Hotswap_MX_1.00u, F.Cu at (28.5, 114.0)
- added SW_1_R1C6: Keyswitch, ScottoKeebs_Hotswap:Hotswap_MX_1.00u, F.Cu at (28.5, 133.0)
- added SW_1_R1C7: Keyswitch, ScottoKeebs_Hotswap:Hotswap_MX_1.00u, F.Cu at (28.5, 152.0)
- added SW_1_R1C8: Keyswitch, ScottoKeebs_Hotswap:Hotswap_MX_1.00u, F.Cu at (28.5, 171.0)
- added SW_1_R1C9: Keyswitch, ScottoKeebs_Hotswap:Hotswap_MX_1.00u, F.Cu at (28.5, 190.0)
- added SW_2_R2C0: Keyswitch, ScottoKeebs_Hotswap:Hotswap_MX_1.00u, F.Cu at (47.5, 9.50)
- added SW_2_R2C1: Keyswitch, ScottoKeebs_Hotswap:Hotswap_MX_1.00u, F.Cu at (47.5, 28.5)
- added SW_2_R2C10: Keyswitch, ScottoKeebs_Hotswap:Hotswap_MX_1.00u, F.Cu at (47.5, 199.5)
- added SW_2_R2C11: Keyswitch, ScottoKeebs_Hotswap:Hotswap_MX_1.00u, F.Cu at (47.5, 218.5)
- added SW_2_R2C12: Keyswitch, ScottoKeebs_Hotswap:Hotswap_MX_1.00u, F.Cu at (47.5, 237.5)
- added SW_2_R2C13: Keyswitch, ScottoKeebs_Hotswap:Hotswap_MX_1.00u, F.Cu at (47.5, 256.5)
- added SW_2_R2C14: Keyswitch, ScottoKeebs_Hotswap:Hotswap_MX_1.00u, F.Cu at (47.5, 275.5)
- added SW_2_R2C15: Keyswitch, ScottoKeebs_Hotswap:Hotswap_MX_1.00u, F.Cu at (47.5, 294.5)
- added SW_2_R2C16: Keyswitch, ScottoKeebs_Hotswap:Hotswap_MX_1.00u, F.Cu at (47.5, 313.5)
- added SW_2_R2C2: Keyswitch, ScottoKeebs_Hotswap:Hotswap_MX_1.00u, F.Cu at (47.5, 47.5)
- added SW_2_R2C3: Keyswitch, ScottoKeebs_Hotswap:Hotswap_MX_1.00u, F.Cu at (47.5, 66.5)
- added SW_2_R2C4: Keyswitch, ScottoKeebs_Hotswap:Hotswap_MX_1.00u, F.Cu at (47.5, 85.5)
- added SW_2_R2C5: Keyswitch, ScottoKeebs_Hotswap:Hotswap_MX_1.00u, F.Cu at (47.5, 104.5)
- added SW_2_R2C6: Keyswitch, ScottoKeebs_Hotswap:Hotswap_MX_1.00u, F.Cu at (47.5, 123.5)
- added SW_2_R2C7: Keyswitch, ScottoKeebs_Hotswap:Hotswap_MX_1.00u, F.Cu at (47.5, 142.5)
- added SW_2_R2C8: Keyswitch, ScottoKeebs_Hotswap:Hotswap_MX_1.00u, F.Cu at (47.5, 161.5)
- added SW_2_R2C9: Keyswitch, ScottoKeebs_Hotswap:Hotswap_MX_1.00u, F.Cu at (47.5, 180.5)
- added SW_3_R0C0: Keyswitch, ScottoKeebs_Hotswap:Hotswap_MX_1.00u, F.Cu at (66.5, 19.0)
- added SW_3_R0C1: Keyswitch, ScottoKeebs_Hotswap:Hotswap_MX_1.00u, F.Cu at (66.5, 38.0)
- added SW_3_R0C10: Keyswitch, ScottoKeebs_Hotswap:Hotswap_MX_1.00u, F.Cu at (66.5, 209.0)
- added SW_3_R0C11: Keyswitch, ScottoKeebs_Hotswap:Hotswap_MX_1.00u, F.Cu at (66.5, 228.0)
- added SW_3_R0C12: Keyswitch, ScottoKeebs_Hotswap:Hotswap_MX_1.00u, F.Cu at (66.5, 247.0)
- added SW_3_R0C13: Keyswitch, ScottoKeebs_Hotswap:Hotswap_MX_1.00u, F.Cu at (66.5, 266.0)
- added SW_3_R0C14: Keyswitch, ScottoKeebs_Hotswap:Hotswap_MX_1.00u, F.Cu at (66.5, 285.0)
- added SW_3_R0C15: Keyswitch, ScottoKeebs_Hotswap:Hotswap_MX_1.00u, F.Cu at (66.5, 304.0)
- added SW_3_R0C2: Keyswitch, ScottoKeebs_Hotswap:Hotswap_MX_1.00u, F.Cu at (66.5, 57.0)
- added SW_3_R0C3: Keyswitch, ScottoKeebs_Hotswap:Hotswap_MX_1.00u, F.Cu at (66.5, 76.0)
- added SW_3_R0C4: Keyswitch, ScottoKeebs_Hotswap:Hotswap_MX_1.00u, F.Cu at (66.5, 95.0)
- added SW_3_R0C5: Keyswitch, ScottoKeebs_Hotswap:Hotswap_MX_1.00u, F.Cu at (66.5, 114.0)
- added SW_3_R0C6: Keyswitch, ScottoKeebs_Hotswap:Hotswap_MX_1.00u, F.Cu at (66.5, 133.0)
- added SW_3_R0C7: Keyswitch, ScottoKeebs_Hotswap:Hotswap_MX_1.00u, F.Cu at (66.5, 152.0)
- added SW_3_R0C8: Keyswitch, ScottoKeebs_Hotswap:Hotswap_MX_1.00u, F.Cu at (66.5, 171.0)
- added SW_3_R0C9: Keyswitch, ScottoKeebs_Hotswap:Hotswap_MX_1.00u, F.Cu at (66.5, 190.0)
- added SW_4_R1C0: Keyswitch, ScottoKeebs_Hotswap:Hotswap_MX_1.00u, F.Cu at (85.5, 9.50)
- added SW_4_R1C1: Keyswitch, ScottoKeebs_Hotswap:Hotswap_MX_1.00u, F.Cu at (85.5, 28.5)
- added SW_4_R1C10: Keyswitch, ScottoKeebs_Hotswap:Hotswap_MX_1.00u, F.Cu at (85.5, 199.5)
- added SW_4_R1C11: Keyswitch, ScottoKeebs_Hotswap:Hotswap_MX_1.00u, F.Cu at (85.5, 218.5)
- added SW_4_R1C12: Keyswitch, ScottoKeebs_Hotswap:Hotswap_MX_1.00u, F.Cu at (85.5, 237.5)
- added SW_4_R1C13: Keyswitch, ScottoKeebs_Hotswap:Hotswap_MX_1.00u, F.Cu at (85.5, 256.5)
- added SW_4_R1C14: Keyswitch, ScottoKeebs_Hotswap:Hotswap_MX_1.00u, F.Cu at (85.5, 275.5)
- added SW_4_R1C15: Keyswitch, ScottoKeebs_Hotswap:Hotswap_MX_1.00u, F.Cu at (85.5, 294.5)
- added SW_4_R1C16: Keyswitch, ScottoKeebs_Hotswap:Hotswap_MX_1.00u, F.Cu at (85.5, 313.5)
- added SW_4_R1C2: Keyswitch, ScottoKeebs_Hotswap:Hotswap_MX_1.00u, F.Cu at (85.5, 47.5)
- added SW_4_R1C3: Keyswitch, ScottoKeebs_Hotswap:Hotswap_MX_1.00u, F.Cu at (85.5, 66.5)
- added SW_4_R1C4: Keyswitch, ScottoKeebs_Hotswap:Hotswap_MX_1.00u, F.Cu at (85.5, 85.5)
- added SW_4_R1C5: Keyswitch, ScottoKeebs_Hotswap:Hotswap_MX_1.00u, F.Cu at (85.5, 104.5)
- added SW_4_R1C6: Keyswitch, ScottoKeebs_Hotswap:Hotswap_MX_1.00u, F.Cu at (85.5, 123.5)
- added SW_4_R1C7: Keyswitch, ScottoKeebs_Hotswap:Hotswap_MX_1.00u, F.Cu at (85.5, 142.5)
- added SW_4_R1C8: Keyswitch, ScottoKeebs_Hotswap:Hotswap_MX_1.00u, F.Cu at (85.5, 161.5)
- added SW_4_R1C9: Keyswitch, ScottoKeebs_Hotswap:Hotswap_MX_1.00u, F.Cu at (85.5, 180.5)
- added SW_5_R2C0: Keyswitch, ScottoKeebs_Hotswap:Hotswap_MX_1.00u, F.Cu at (104.5, 19.0)
- added SW_5_R2C1: Keyswitch, ScottoKeebs_Hotswap:Hotswap_MX_1.00u, F.Cu at (104.5, 38.0)
- added SW_5_R2C10: Keyswitch, ScottoKeebs_Hotswap:Hotswap_MX_1.00u, F.Cu at (104.5, 209.0)
- added SW_5_R2C11: Keyswitch, ScottoKeebs_Hotswap:Hotswap_MX_1.00u, F.Cu at (104.5, 228.0)
- added SW_5_R2C12: Keyswitch, ScottoKeebs_Hotswap:Hotswap_MX_1.00u, F.Cu at (104.5, 247.0)
- added SW_5_R2C13: Keyswitch, ScottoKeebs_Hotswap:Hotswap_MX_1.00u, F.Cu at (104.5, 266.0)
- added SW_5_R2C14: Keyswitch, ScottoKeebs_Hotswap:Hotswap_MX_1.00u, F.Cu at (104.5, 285.0)
- added SW_5_R2C15: Keyswitch, ScottoKeebs_Hotswap:Hotswap_MX_1.00u, F.Cu at (108.3, 306.5)
- added SW_5_R2C2: Keyswitch, ScottoKeebs_Hotswap:Hotswap_MX_1.00u, F.Cu at (104.5, 57.0)
- added SW_5_R2C3: Keyswitch, ScottoKeebs_Hotswap:Hotswap_MX_1.00u, F.Cu at (104.5, 76.0)
- added SW_5_R2C4: Keyswitch, ScottoKeebs_Hotswap:Hotswap_MX_1.00u, F.Cu at (104.5, 95.0)
- added SW_5_R2C5: Keyswitch, ScottoKeebs_Hotswap:Hotswap_MX_1.00u, F.Cu at (104.5, 114.0)
- added SW_5_R2C6: Keyswitch, ScottoKeebs_Hotswap:Hotswap_MX_1.00u, F.Cu at (104.5, 133.0)
- added SW_5_R2C7: Keyswitch, ScottoKeebs_Hotswap:Hotswap_MX_1.00u, F.Cu at (104.5, 152.0)
- added SW_5_R2C8: Keyswitch, ScottoKeebs_Hotswap:Hotswap_MX_1.00u, F.Cu at (104.5, 171.0)
- added SW_5_R2C9: Keyswitch, ScottoKeebs_Hotswap:Hotswap_MX_1.00u, F.Cu at (104.5, 190.0)
- moved A1 276.6 mm to (485.7, 46.7), turned to 0 degrees
Connections:
- A1 pad 10: Column 5 -> Column 12
- A1 pad 11: Column 6 -> Column 13
- A1 pad 12: Column 7 -> Column 14
- A1 pad 13: Column 8 -> Column 15
- A1 pad 14: Column 9 -> Column 16
- A1 pad 15: Row 0 -> Column 0
- A1 pad 16: Row 1 -> Column 1
- A1 pad 17: Row 2 -> Column 2
- A1 pad 18: Row 3 -> Column 3
- A1 pad 19: Row 4 -> Column 4
- A1 pad 20: Row 5 -> Column 5
- A1 pad 21: Row 6 -> Column 6
- A1 pad 22: Row 7 -> Column 7
- A1 pad 23: Row 8 -> Column 8
- A1 pad 24: Row 9 -> Column 9
- A1 pad 25: Column 0 -> Column 10
- A1 pad 26: Column 1 -> Row 0
- A1 pad 27: Column 2 -> Row 1
- A1 pad 28: Column 3 -> Row 2
- A1 pad 9: Column 4 -> Column 11

Commit message: teste, pcb, esquema
codigo de teste criado;
atualizaçoes no pcb e esquema.
Parts:
- moved A1 707.8 mm to (-77.9, 475.0), turned to 180 degrees
- moved D_R0C0 528.9 mm to (0.00, 28.5)
- moved SW_0_R0C0 13.4 mm to (19.0, 19.0), turned to -90 degrees
- moved SW_0_R0C1 13.4 mm to (19.0, 38.0), turned to -90 degrees
- moved SW_0_R0C10 13.4 mm to (19.0, 209.0)
- moved SW_0_R0C11 13.4 mm to (19.0, 228.0)
- moved SW_0_R0C12 13.4 mm to (19.0, 247.0)
- moved SW_0_R0C13 13.4 mm to (19.0, 266.0)
- moved SW_0_R0C14 13.4 mm to (19.0, 285.0)
- moved SW_0_R0C15 13.4 mm to (19.0, 304.0)
- moved SW_0_R0C16 13.4 mm to (19.0, 323.0)
- moved SW_0_R0C2 13.4 mm to (19.0, 57.0)
- moved SW_0_R0C3 13.4 mm to (19.0, 76.0)
- moved SW_0_R0C4 13.4 mm to (19.0, 95.0)
- moved SW_0_R0C5 13.4 mm to (19.0, 114.0)
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Routing:
- net Column 1: track 0.00 -> 114.7 mm
- net Column 0: track 0.00 -> 114.7 mm
- net Net-(D_R0C0-A): track 0.00 -> 60.9 mm

Commit message: octave adjust
Parts:
- added SW_1_R1C16: Keyswitch, ScottoKeebs_Hotswap:Hotswap_MX_1.00u, F.Cu at (49.7, 391.8)
- added SW_3_R0C16: Keyswitch, ScottoKeebs_Hotswap:Hotswap_MX_1.00u, F.Cu at (87.7, 391.8)
- added SW_5_R2C16: Keyswitch, ScottoKeebs_Hotswap:Hotswap_MX_1.00u, F.Cu at (125.7, 391.8)
- A1, D_R0C0, D_R0C1, D_R0C10, D_R0C11, D_R0C12, D_R0C13, D_R0C14, D_R0C15, D_R0C16, D_R0C2, D_R0C3, D_R0C4, D_R0C5, D_R0C6, D_R0C7, D_R0C8, D_R0C9, D_R1C0, D_R1C1, D_R1C10, D_R1C11, D_R1C12, D_R1C13, D_R1C14, D_R1C15, D_R1C16, D_R1C2, D_R1C3, D_R1C4, D_R1C5, D_R1C6, D_R1C7, D_R1C8, D_R1C9, D_R2C0, D_R2C1, D_R2C10, D_R2C11, D_R2C12, D_R2C13, D_R2C14, D_R2C15, D_R2C16, D_R2C2, D_R2C3, D_R2C4, D_R2C5, D_R2C6, D_R2C7, D_R2C8, D_R2C9: moved to B.Cu
- moved D_R0C16 619.1 mm to (21.4, 391.9)
- moved D_R0C15 610.8 mm to (21.4, 372.9)
- moved D_R1C16 609.6 mm to (40.4, 401.4)
- moved D_R0C14 602.6 mm to (21.5, 353.9)
- moved D_R1C15 601.5 mm to (40.1, 382.4)
- moved D_R0C13 595.0 mm to (21.4, 334.9)
- moved D_R1C14 593.5 mm to (40.1, 363.4)
- moved D_R2C16 589.9 mm to (59.4, 391.9)
- moved D_R1C13 585.7 mm to (40.1, 344.4)
- moved D_R2C15 582.4 mm to (58.9, 372.9)
- moved D_R1C12 578.3 mm to (40.1, 325.4)
- moved D_R2C14 574.5 mm to (59.1, 353.9)
- moved D_R1C11 571.2 mm to (40.1, 306.4)
- moved D_R2C13 567.1 mm to (59.1, 334.9)
- moved D_R1C10 564.4 mm to (40.1, 287.4)
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Connections:
- A1 pad 15: Column 0 -> Row 0
- A1 pad 16: Column 1 -> Column 0
- A1 pad 17: Column 2 -> Column 1
- A1 pad 18: Column 3 -> Column 10
- A1 pad 19: Column 4 -> Column 9
- A1 pad 20: Column 5 -> Column 8
- A1 pad 21: Column 6 -> Column 7
- A1 pad 22: Column 7 -> Column 6
- A1 pad 23: Column 8 -> Column 5
- A1 pad 24: Column 9 -> Column 4
- A1 pad 25: Column 10 -> Column 3
- A1 pad 26: Row 0 -> Column 2
Routing:
- net Row 1: track 0.00 -> 345.2 mm
- net Row 0: track 0.00 -> 330.3 mm
- net Row 2: track 0.00 -> 329.9 mm
- net Column 1: track 114.7 -> 0.00 mm
- net Net-(D_R0C0-A): track 60.9 -> 8.33 mm
- net Column 0: track 114.7 -> 128.8 mm
- net Net-(D_R2C2-A): track 0.00 -> 8.57 mm
- net Net-(D_R2C1-A): track 0.00 -> 8.57 mm
- net Net-(D_R2C0-A): track 0.00 -> 8.57 mm
- net Net-(D_R1C0-A): track 0.00 -> 8.33 mm
- net Net-(D_R0C1-A): track 0.00 -> 8.33 mm
- net Net-(D_R1C1-A): track 0.00 -> 8.08 mm
- net (no net): track 0.00 -> 4.05 mm
