File: kicad_project/Chromatic.kicad_pcb (KiCad board)
At the start: 2 copper layers, 159 parts, among them J1 J1, J2 J2

Commit message: arrumado
Parts:
- SW_0_R0C0, SW_0_R0C1, SW_0_R0C10, SW_0_R0C11, SW_0_R0C12, SW_0_R0C13, SW_0_R0C14, SW_0_R0C15, SW_0_R0C16, SW_0_R0C2, SW_0_R0C3, SW_0_R0C4, SW_0_R0C5, SW_0_R0C6, SW_0_R0C7, SW_0_R0C8, SW_0_R0C9, SW_1_R1C0, SW_1_R1C1, SW_1_R1C10, SW_1_R1C11, SW_1_R1C12, SW_1_R1C13, SW_1_R1C14, SW_1_R1C15, SW_1_R1C16, SW_1_R1C2, SW_1_R1C3, SW_1_R1C4, SW_1_R1C5, SW_1_R1C6, SW_1_R1C7, SW_1_R1C8, SW_1_R1C9, SW_2_R2C0, SW_2_R2C1, SW_2_R2C10, SW_2_R2C11, SW_2_R2C12, SW_2_R2C13, SW_2_R2C14, SW_2_R2C15, SW_2_R2C16, SW_2_R2C2, SW_2_R2C3, SW_2_R2C4, SW_2_R2C5, SW_2_R2C6, SW_2_R2C7, SW_2_R2C8, SW_2_R2C9, SW_3_R0C0, SW_3_R0C1, SW_3_R0C10, SW_3_R0C11, SW_3_R0C12, SW_3_R0C13, SW_3_R0C14, SW_3_R0C15, SW_3_R0C16, SW_3_R0C2, SW_3_R0C3, SW_3_R0C4, SW_3_R0C5, SW_3_R0C6, SW_3_R0C7, SW_3_R0C8, SW_3_R0C9, SW_4_R1C0, SW_4_R1C1, SW_4_R1C10, SW_4_R1C11, SW_4_R1C12, SW_4_R1C13, SW_4_R1C14, SW_4_R1C15, SW_4_R1C16, SW_4_R1C2, SW_4_R1C3, SW_4_R1C4, SW_4_R1C5, SW_4_R1C6, SW_4_R1C7, SW_4_R1C8, SW_4_R1C9, SW_5_R2C0, SW_5_R2C1, SW_5_R2C10, SW_5_R2C11, SW_5_R2C12, SW_5_R2C13, SW_5_R2C14, SW_5_R2C15, SW_5_R2C16, SW_5_R2C2, SW_5_R2C3, SW_5_R2C4, SW_5_R2C5, SW_5_R2C6, SW_5_R2C7, SW_5_R2C8, SW_5_R2C9: moved to B.Cu
- moved SW_5_R2C12 555.5 mm to (6.07, 187.0)
- moved SW_5_R2C13 547.9 mm to (6.07, 171.4)
- moved SW_5_R2C14 542.0 mm to (6.07, 155.9)
- moved SW_5_R2C15 537.8 mm to (6.07, 140.3)
- moved SW_5_R2C16 535.4 mm to (6.07, 124.8)
- moved SW_4_R1C12 524.6 mm to (-27.2, 78.1)
- moved SW_4_R1C15 521.8 mm to (-27.2, 31.5)
- moved SW_4_R1C13 521.3 mm to (-27.2, 62.6)
- moved SW_4_R1C14 520.6 mm to (-27.2, 47.0)
- moved SW_4_R1C16 512.2 mm to (-10.6, 202.5)
- moved SW_2_R2C12 492.5 mm to (-132.1, 108.7)
- moved SW_3_R0C12 489.9 mm to (-43.8, 155.9)
- moved SW_2_R2C13 488.9 mm to (-132.1, 93.2)
- moved SW_3_R0C13 483.2 mm to (-43.8, 140.3)
- moved SW_3_R0C14 478.5 mm to (-43.8, 124.8)
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