File: kicad_project/Chromatic.kicad_pcb (KiCad board)
At the start: 2 copper layers, 159 parts, among them J1 J1, J2 J2

Commit message: LAYOUT OK
Parts:
- A3, D_R0C12, D_R0C13, D_R0C14, D_R0C15, D_R0C16, D_R1C12, D_R1C13, D_R1C14, D_R1C15, D_R1C16, D_R2C12, D_R2C13, D_R2C14, D_R2C15, D_R2C16, R0, R1, R2: moved to B.Cu
- SW_0_R0C12, SW_0_R0C13, SW_0_R0C14, SW_0_R0C15, SW_0_R0C16, SW_1_R1C12, SW_1_R1C13, SW_1_R1C14, SW_1_R1C15, SW_1_R1C16, SW_2_R2C12, SW_2_R2C13, SW_2_R2C14, SW_2_R2C15, SW_2_R2C16, SW_3_R0C12, SW_3_R0C13, SW_3_R0C14, SW_3_R0C15, SW_3_R0C16, SW_4_R1C12, SW_4_R1C13, SW_4_R1C14, SW_4_R1C15, SW_4_R1C16, SW_5_R2C12, SW_5_R2C13, SW_5_R2C14, SW_5_R2C15, SW_5_R2C16: moved to F.Cu
- moved D_R1C16 612.9 mm to (43.3, 417.2), turned to 180 degrees
- moved D_R0C16 612.2 mm to (24.3, 407.7), turned to 180 degrees
- moved D_R1C15 600.2 mm to (43.3, 398.2), turned to 180 degrees
- moved D_R0C15 599.4 mm to (24.3, 388.7), turned to 180 degrees
- moved D_R2C16 598.3 mm to (62.3, 407.7), turned to 180 degrees
- moved D_R1C14 587.6 mm to (43.3, 379.2), turned to 180 degrees
- moved D_R0C14 586.6 mm to (24.3, 369.7), turned to 180 degrees
- moved D_R2C15 585.8 mm to (62.3, 388.7), turned to 180 degrees
- moved D_R1C13 575.1 mm to (43.3, 360.2), turned to 180 degrees
- moved D_R0C13 574.1 mm to (24.3, 350.7), turned to 180 degrees
- moved D_R2C14 573.6 mm to (62.3, 369.7), turned to 180 degrees
- moved D_R1C12 562.7 mm to (43.1, 341.2), turned to 180 degrees
- moved D_R2C13 561.5 mm to (62.3, 350.7), turned to 180 degrees
- moved D_R2C12 550.7 mm to (62.9, 332.6), turned to 180 degrees
- moved D_R0C12 532.8 mm to (23.9, 332.6), turned to 180 degrees
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Routing:
- net Net-(J2-Pin_5): track 0.00 -> 173.6 mm
- net Net-(J2-Pin_4): track 0.00 -> 173.6 mm
- net Net-(J2-Pin_2): track 0.00 -> 172.1 mm
- net Net-(J2-Pin_1): track 0.00 -> 171.7 mm
- net Net-(J2-Pin_3): track 0.00 -> 170.2 mm
- net Net-(D_R2C12-A): track 0.00 -> 77.3 mm
- net Net-(D_R1C16-A): track 0.00 -> 67.1 mm
- net Net-(D_R1C12-A): track 0.00 -> 67.1 mm
- net Net-(D_R2C14-A): track 0.00 -> 67.1 mm
- net Net-(D_R2C16-A): track 0.00 -> 66.9 mm
- net Net-(D_R1C15-A): track 0.00 -> 66.8 mm
- net Net-(D_R1C13-A): track 0.00 -> 66.7 mm
- net Net-(D_R1C14-A): track 0.00 -> 66.3 mm
- net Net-(D_R2C13-A): track 0.00 -> 65.3 mm
- net Net-(D_R2C15-A): track 0.00 -> 65.2 mm
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
Commit message: footprint
Parts:
- A3: moved to F.Cu
- J1, J2: moved to B.Cu
- moved J2 272.0 mm to (150.0, 357.2), turned to 180 degrees
- moved A3 53.8 mm to (130.8, 0.60)
- moved J1 8.66 mm to (144.2, 298.4), turned to 90 degrees
Connections:
- A3 pad A3: Column 15 -> Row 2
- A3 pad A4: Column 16 -> Row 1
- A3 pad A5: Column 11 -> Row 0
- A3 pad D0: Row 1 -> unconnected-(A3-D0/RX-PadD0)
- A3 pad D1: Row 0 -> unconnected-(A3-D1/TX-PadD1)
- A3 pad D13: Row 2 -> unconnected-(A3-PadD13)
Routing:
- net Row 0: track 0.00 -> 46.9 mm
- net Row 1: track 0.00 -> 45.6 mm
- net Row 2: track 0.00 -> 4.14 mm
