File: kicad_project/Chromatic.kicad_pcb (KiCad board)
At the start: 2 copper layers, 159 parts, among them J1 J1, J2 J2

Commit message: done
Parts:
- moved D_R1C10 37.6 mm to (78.9, 279.6)
- moved D_R1C9 37.6 mm to (78.9, 260.6)
- moved D_R0C1 37.6 mm to (59.6, 99.1)
- moved D_R0C10 37.6 mm to (59.6, 270.1)
- moved D_R0C11 37.6 mm to (59.9, 289.1)
- moved D_R0C2 37.6 mm to (59.6, 118.1)
- moved D_R1C1 37.6 mm to (78.9, 108.7)
- moved D_R1C3 37.6 mm to (78.9, 146.7)
- moved D_R1C4 37.6 mm to (78.9, 165.7)
- moved D_R1C5 37.6 mm to (78.9, 184.7)
- moved D_R1C6 37.6 mm to (78.9, 203.7)
- moved D_R1C7 37.6 mm to (78.9, 222.7)
- moved D_R1C8 37.6 mm to (78.9, 241.7)
- moved D_R2C0 37.6 mm to (97.4, 80.2)
- moved D_R2C1 37.6 mm to (97.4, 99.2)
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Routing:
- net Net-(J2-Pin_5): track 208.7 -> 204.3 mm
- net Net-(D_R2C12-A): track 77.3 -> 79.6 mm
- net Column 8: track 377.5 -> 379.0 mm
- net Column 10: track 421.4 -> 423.0 mm
- net Net-(D_R1C12-K): track 165.9 -> 164.5 mm
- net Net-(D_R2C12-K): track 151.5 -> 150.3 mm
- net Net-(D_R1C12-A): track 67.1 -> 68.1 mm
- net Net-(J2-Pin_4): track 211.8 -> 211.1 mm
- net Net-(J2-Pin_1): track 259.5 -> 258.9 mm
- net Net-(J2-Pin_2): track 237.9 -> 237.3 mm
- net Net-(D_R0C12-K): track 193.7 -> 193.1 mm
