File: kicad_project/Chromatic.kicad_sch (KiCad schematic)
At the start: 159 parts, among them J1 J1, J2 J2

Commit message: footprint
Parts:
- A3: footprint arduino-library:Arduino_Leonardo_Shield -> Leonardo_Rev3e:1X06
Connections:
- net Column 11: no longer A3.A5
- net Column 15: no longer A3.A3
- net Column 16: no longer A3.A4
- net Row 0: now also A3.A5; no longer A3.D1 (D1/TX)
- net Row 1: now also A3.A4; no longer A3.D0 (D0/RX)
- net Row 2: now also A3.A3; no longer A3.D13
Changed lines of the file:
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@@
 		)
 	)
-	(global_label "Column 4"
+	(global_label "Column 16"
 		(shape input)
-		(at 146.05 35.56 90)
+		(at 85.09 110.49 180)
 		(fields_autoplaced yes)
 		(effects
@@
 				(size 1.27 1.27)
 			)
-			(justify left)
+			(justify right)
 		)
 		(property "Intersheetrefs" "${INTERSHEET_REFS}"
-			(at 146.05 23.3222 90)
+			(at 71.6427 110.49 0)
 			(hide yes)
 			(show_name no)
@@
 					(size 1.27 1.27)
 				)
-				(justify left)
+				(justify right)
 			)
 		)
 	)
-	(global_label "Column 5"
+	(global_label "Column 11"
 		(shape input)
-		(at 156.21 35.56 90)
+		(at 85.09 107.95 180)
+		(fields_autoplaced yes)
+		(effects
+			(font
+				(size 1.27 1.27)
+			)
+			(justify right)
+		)
+		(property "Intersheetrefs" "${INTERSHEET_REFS}"
+			(at 71.6427 107.95 0)
+			(hide yes)
+			(show_name no)
+			(do_not_autoplace no)
+			(effects
+				(font
+					(size 1.27 1.27)
+				)
+				(justify right)
+			)
+		)
+	)
+	(global_label "Column 4"
+		(shape input)
+		(at 146.05 35.56 90)
 		(fields_autoplaced yes)
 		(effects
@@
 		)
 		(property "Intersheetrefs" "${INTERSHEET_REFS}"
-			(at 156.21 23.3222 90)
+			(at 146.05 23.3222 90)
 			(hide yes)
 			(show_name no)
@@
 		)
 	)
-	(global_label "D_R1C11"
+	(global_label "Column 5"
 		(shape input)
-		(at 224.79 53.34 0)
+		(at 156.21 35.56 90)
 		(fields_autoplaced yes)
 		(effects
@@
 		)
 		(property "Intersheetrefs" "${INTERSHEET_REFS}"
-			(at 236.1813 53.34 0)
+			(at 156.21 23.3222 90)
 			(hide yes)
 			(show_name no)
@@
 		)
 	)
-	(global_label "Column 16"
+	(global_label "D_R1C11"
 		(shape input)
-		(at 16.51 86.36 180)
+		(at 224.79 53.34 0)
 		(fields_autoplaced yes)
 		(effects
@@
 				(size 1.27 1.27)
 			)
-			(justify right)
+			(justify left)
 		)
 		(property "Intersheetrefs" "${INTERSHEET_REFS}"
-			(at 3.0627 86.36 0)
+			(at 236.1813 53.34 0)
 			(hide yes)
 			(show_name no)
@@
 					(size 1.27 1.27)
 				)
-				(justify right)
+				(justify left)
 			)
 		)
@@
 		)
 	)
-	(global_label "Row 0"
+	(global_label "Column 5"
 		(shape input)
-		(at 16.51 68.58 180)
+		(at 67.31 78.74 0)
 		(fields_autoplaced yes)
 		(effects
@@
 				(size 1.27 1.27)
 			)
-			(justify right)
+			(justify left)
 		)
 		(property "Intersheetrefs" "${INTERSHEET_REFS}"
-			(at 7.5982 68.58 0)
+			(at 79.5478 78.74 0)
 			(hide yes)
 			(show_name no)
@@
 					(size 1.27 1.27)
 				)
-				(justify right)
+				(justify left)
 			)
 		)
 	)
-	(global_label "Column 5"
+	(global_label "Row 0"
 		(shape input)
-		(at 67.31 78.74 0)
+		(at 16.51 83.82 180)
 		(fields_autoplaced yes)
 		(effects
@@
 				(size 1.27 1.27)
 			)
-			(justify left)
+			(justify right)
 		)
 		(property "Intersheetrefs" "${INTERSHEET_REFS}"
-			(at 79.5478 78.74 0)
+			(at 7.5982 83.82 0)
 			(hide yes)
 			(show_name no)
@@
 					(size 1.27 1.27)
 				)
-				(justify left)
+				(justify right)
 			)
 		)
@@
 		)
 	)
-	(global_label "Row 2"
-		(shape input)
-		(at 67.31 93.98 0)
-		(fields_autoplaced yes)
-		(effects
-			(font
-				(size 1.27 1.27)
-			)
-			(justify left)
-		)
-		(property "Intersheetrefs" "${INTERSHEET_REFS}"
-			(at 76.2218 93.98 0)
-			(hide yes)
-			(show_name no)
-			(do_not_autoplace no)
-			(effects
-				(font
-					(size 1.27 1.27)
-				)
-				(justify left)
-			)
-		)
-	)
 	(global_label "Column 12"
 		(shape input)
@@
 		)
 	)
-	(global_label "Column 15"
+	(global_label "Row 2"
 		(shape input)
 		(at 16.51 88.9 180)
@@
 		)
 		(property "Intersheetrefs" "${INTERSHEET_REFS}"
-			(at 3.0627 88.9 0)
+			(at 7.5982 88.9 0)
 			(hide yes)
 			(show_name no)
@@
 		)
 	)
-	(global_label "Column 0"
+	(global_label "Column 15"
 		(shape input)
-		(at 105.41 35.56 90)
+		(at 85.09 113.03 180)
 		(fields_autoplaced yes)
 		(effects
@@
 				(size 1.27 1.27)
 			)
-			(justify left)
+			(justify right)
 		)
 		(property "Intersheetrefs" "${INTERSHEET_REFS}"
-			(at 105.41 23.3222 90)
+			(at 71.6427 113.03 0)
 			(hide yes)
 			(show_name no)
@@
 					(size 1.27 1.27)
 				)
-				(justify left)
+				(justify right)
 			)
 		)
 	)
-	(global_label "Pin 8"
+	(global_label "Column 0"
 		(shape input)
-		(at 124.46 114.3 0)
+		(at 105.41 35.56 90)
 		(fields_autoplaced yes)
 		(effects
@@
 		)
 		(property "Intersheetrefs" "${INTERSHEET_REFS}"
-			(at 132.6461 114.3 0)
+			(at 105.41 23.3222 90)
 			(hide yes)
 			(show_name no)
@@
 		)
 	)
-	(global_label "Column 2"
+	(global_label "Pin 8"
 		(shape input)
-		(at 125.73 35.56 90)
+		(at 124.46 114.3 0)
 		(fields_autoplaced yes)
 		(effects
@@
 		)
 		(property "Intersheetrefs" "${INTERSHEET_REFS}"
-			(at 125.73 23.3222 90)
+			(at 132.6461 114.3 0)
 			(hide yes)
 			(show_name no)
@@
 		)
 	)
-	(global_label "Row 1"
+	(global_label "Column 2"
 		(shape input)
-		(at 16.51 66.04 180)
+		(at 125.73 35.56 90)
 		(fields_autoplaced yes)
 		(effects
@@
 				(size 1.27 1.27)
 			)
-			(justify right)
+			(justify left)
 		)
 		(property "Intersheetrefs" "${INTERSHEET_REFS}"
-			(at 7.5982 66.04 0)
+			(at 125.73 23.3222 90)
 			(hide yes)
 			(show_name no)
@@
 					(size 1.27 1.27)
 				)
-				(justify right)
+				(justify left)
 			)
 		)
@@
 		)
 	)
-	(global_label "Column 11"
-		(shape input)
-		(at 16.51 83.82 180)
-		(fields_autoplaced yes)
-		(effects
-			(font
-				(size 1.27 1.27)
-			)
-			(justify right)
-		)
-		(property "Intersheetrefs" "${INTERSHEET_REFS}"
-			(at 3.0627 83.82 0)
-			(hide yes)
-			(show_name no)
-			(do_not_autoplace no)
-			(effects
-				(font
-					(size 1.27 1.27)
-				)
-				(justify right)
-			)
-		)
-	)
 	(global_label "D_R0C11"
 		(shape input)
@@
 		)
 	)
+	(global_label "Row 1"
+		(shape input)
+		(at 16.51 86.36 180)
+		(fields_autoplaced yes)
+		(effects
+			(font
+				(size 1.27 1.27)
+			)
+			(justify right)
+		)
+		(property "Intersheetrefs" "${INTERSHEET_REFS}"
+			(at 7.5982 86.36 0)
+			(hide yes)
+			(show_name no)
+			(do_not_autoplace no)
+			(effects
+				(font
+					(size 1.27 1.27)
+				)
+				(justify right)
+			)
+		)
+	)
 	(symbol
 		(lib_id "ScottoKeebs:Placeholder_Keyswitch")
@@
 			)
 		)
-		(property "Footprint" "arduino-library:Arduino_Leonardo_Shield"
+		(property "Footprint" "Leonardo_Rev3e:1X06"
 			(at 41.91 130.81 0)
 			(hide yes)
